File: RGB_Driver.brd (EAGLE design)
At the start: 54.9 x 28 mm, 8 parts, among them Q1 TIP41C, Q2 TIP41C, Q3 TIP41C, X1 1751277, X2 1751264

Commit message: Add files via upload
- Add header pins
- Add fuse
- Add 2 slot terminal block
- Remove 5 slot terminal block
Parts:
- removed X2: 1751264, con-phoenix-350:1751264
- added F1: (no value), fuse:SHK20L
- added JP1: (no value), pinhead:1X03
- added X3: 1751248, con-phoenix-350:1751248
- X1: value 1751277 -> 1751264; device con-phoenix-350:1751277 -> con-phoenix-350:1751264
- moved X1 40.5 mm to (48.8, 14.0), turned to 90 degrees
- moved R1 5.75 mm to (16.3, 12.6)
- moved R2 5.38 mm to (16.2, 8.85)
- moved R3 4.78 mm to (16.3, 5.26)
- moved Q1 4.41 mm to (28.5, 9.86)
- moved Q2 4.40 mm to (35.6, 10.0)
- moved Q3 4.32 mm to (42.5, 9.90)
Connections:
- new net N$10: F1.2A, X1.4
- net +12V: now also F1.1A, X3.1; no longer X1.1, X2.4
- net GND: now also X3.2; no longer X1.2
- net N$4: now also X1.3; no longer X2.3
- net N$5: now also X1.2; no longer X2.2
- net N$6: now also X1.1; no longer X2.1
- net N$7: now also JP1.3; no longer X1.5
- net N$8: now also JP1.2; no longer X1.4
- net N$9: now also JP1.1; no longer X1.3
Routing:
- net +12V: track 41.1 -> 7.51 mm
- net N$10: track 0.00 -> 13.5 mm
- net N$4: track 38.5 -> 29.9 mm, vias 0 -> 1
- net N$3: track 31.6 -> 26.6 mm
- net N$9: track 7.35 -> 5.18 mm
- net N$5: track 21.5 -> 19.4 mm
- net N$2: track 20.9 -> 22.4 mm
- net N$1: track 4.63 -> 5.93 mm
- net N$8: track 6.56 -> 5.32 mm
- net N$6: track 10.4 -> 9.41 mm
Other:
- board text added: "1.5 Amps MAX"
- board text added: "1K Ω"
- board text added: "RGB_Driver V3"
- board text removed: "RGB_Driver V2.1"
