File: RGB_Driver.sch (EAGLE design)
At the start: 8 parts, among them Q1 TIP41C, Q2 TIP41C, Q3 TIP41C, X1 1751277, X2 1751264

Commit message: Add files via upload
- Add header pins
- Add fuse
- Add 2 slot terminal block
- Remove 5 slot terminal block
Parts:
- removed X2: 1751264, con-phoenix-350:1751264
- added F1: (no value), fuse:SHK20L
- added JP1: (no value), pinhead:PINHD-1X3
- added X3: 1751248, con-phoenix-350:1751248
- X1: value 1751277 -> 1751264; device con-phoenix-350:1751277 -> con-phoenix-350:1751264
Connections:
- new net N$10: F1.2A, X1-4.K
- net +12V: now also F1.1A, X3-1.K; no longer X1-1.K, X2-4.K
- net GND: now also X3-2.K; no longer X1-2.K
- net N$4: now also X1-3.K; no longer X2-3.K
- net N$5: now also X1-2.K; no longer X2-2.K
- net N$6: now also X1-1.K; no longer X2-1.K
- net N$7: now also JP1.3; no longer X1-5.K
- net N$8: now also JP1.2; no longer X1-4.K
- net N$9: now also JP1.1; no longer X1-3.K
Other:
- moved on the sheet: X1-1, X1-2, X1-3, X1-4
